File: _autosave-cts_switchpcb.kicad_pcb (KiCad board)
At the start: 2 copper layers, 47.8 x 28.1 mm, 13 parts, among them J2 Conn_01x06, SW1 SW_SPDT, SW2 SW_SPDT, SW3 SW_SPDT, SW4 SW_SPDT

Commit message: Skibidi toilet
Parts:
- removed D1, D2: LED, LED_SMD:LED_0201_0603Metric
- removed R1, R2: R, Resistor_SMD:R_0201_0603Metric
- moved H3 22.7 mm to (89.5, 75.5)
- moved H4 20.0 mm to (110.8, 75.2)
- moved H2 20.0 mm to (110.8, 54.0)
- moved H1 12.2 mm to (89.5, 54.0)
Routing:
- added copper zone on B.Cu, net GND
Other:
- board size 47.8 x 28.1 mm -> 27.8 x 28.1 mm
